File: hardware/ao-4u-4i.kicad_pcb (KiCad board)
At the start: 4 copper layers, 100 x 85 mm, 225 parts, among them J101 TNG-Power-TOP, J102 TNG-Power-BTM, J103 TNG-Data-TOP, J104 TNG-Data-BTM, P102 Debug, P103 PE, P201 INPUT0, P202 INPUT1, P203 INPUT2, P204 INPUT3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

Commit message: change esd diodes
Parts:
- D211, D212, D215, D216, D219, D220, D223, D224: value DESD1P0RFW -> CDSOT23-T12C
Changed lines of the file:
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@@
     (1 GND power hide)
     (2 VCC power hide)
-    (31 B.Cu signal)
+    (31 B.Cu signal hide)
     (32 B.Adhes user)
     (33 F.Adhes user hide)
@@
     (aux_axis_origin 89.8 62.5)
     (grid_origin 89.8 62.5)
-    (visible_elements FFFFFF7F)
+    (visible_elements FFFEFF7F)
     (pcbplotparams
       (layerselection 0x010fc_ffffffff)
@@
       (effects (font (size 0.3 0.3) (thickness 0.075)))
     )
-    (fp_text value DESD1P0RFW (at 0 -0.25 90) (layer F.Fab)
+    (fp_text value CDSOT23-T12C (at 0 -0.25 90) (layer F.Fab)
       (effects (font (size 0.29972 0.29972) (thickness 0.07112)))
     )
@@
       (effects (font (size 0.3 0.3) (thickness 0.075)))
     )
-    (fp_text value DESD1P0RFW (at -0.65 -0.3 90) (layer F.Fab)
+    (fp_text value CDSOT23-T12C (at -0.65 -0.3 90) (layer F.Fab)
       (effects (font (size 0.29972 0.29972) (thickness 0.07112)))
     )
@@
       (effects (font (size 0.3 0.3) (thickness 0.075)))
     )
-    (fp_text value DESD1P0RFW (at 0 -0.25 90) (layer F.Fab)
+    (fp_text value CDSOT23-T12C (at 0 -0.25 90) (layer F.Fab)
       (effects (font (size 0.29972 0.29972) (thickness 0.07112)))
     )
@@
       (effects (font (size 0.3 0.3) (thickness 0.075)))
     )
-    (fp_text value DESD1P0RFW (at -0.65 -0.3) (layer F.Fab)
+    (fp_text value CDSOT23-T12C (at -0.65 -0.3) (layer F.Fab)
       (effects (font (size 0.29972 0.29972) (thickness 0.07112)))
     )
@@
       (effects (font (size 0.3 0.3) (thickness 0.075)))
     )
-    (fp_text value DESD1P0RFW (at 0 -0.3 180) (layer F.Fab)
+    (fp_text value CDSOT23-T12C (at 0 -0.3 180) (layer F.Fab)
       (effects (font (size 0.29972 0.29972) (thickness 0.07112)))
     )
@@
       (effects (font (size 0.3 0.3) (thickness 0.075)))
     )
-    (fp_text value DESD1P0RFW (at -0.65 -0.3 90) (layer F.Fab)
+    (fp_text value CDSOT23-T12C (at -0.65 -0.3 90) (layer F.Fab)
       (effects (font (size 0.29972 0.29972) (thickness 0.07112)))
     )
@@
       (effects (font (size 0.3 0.3) (thickness 0.075)))
     )
-    (fp_text value DESD1P0RFW (at -0.65 -0.3) (layer F.Fab)
+    (fp_text value CDSOT23-T12C (at -0.65 -0.3) (layer F.Fab)
       (effects (font (size 0.29972 0.29972) (thickness 0.07112)))
     )
@@
       (effects (font (size 0.3 0.3) (thickness 0.075)))
     )
-    (fp_text value DESD1P0RFW (at -0.65 -0.3) (layer F.Fab)
+    (fp_text value CDSOT23-T12C (at -0.65 -0.3) (layer F.Fab)
       (effects (font (size 0.29972 0.29972) (thickness 0.07112)))
     )

Commit message: fix values
Parts:
- C127, C128: value 4.7nF/2kV -> 1nF/2kV
- R101: value 510 -> 1k

Commit message: specify value
Parts:
- C115: value TBD -> 2.2uF

Commit message: fix diode values
Parts:
- D211, D212, D215, D216, D219, D220, D223, D224: value CDSOT23-T12C -> CDSOT23-T15C
Connections:
- J101 pad 21: (no net) -> Net-(J101-Pad21)
- J101 pad 22: (no net) -> Net-(J101-Pad22)
- J101 pad 23: (no net) -> Net-(J101-Pad23)
- J101 pad 24: (no net) -> Net-(J101-Pad24)
- J101 pad 25: (no net) -> Net-(J101-Pad25)
- J101 pad 26: (no net) -> Net-(J101-Pad26)
- J101 pad 27: (no net) -> Net-(J101-Pad27)
- J101 pad 28: (no net) -> Net-(J101-Pad28)
- J101 pad 29: (no net) -> Net-(J101-Pad29)
- J101 pad 30: (no net) -> Net-(J101-Pad30)
- J102 pad 21: (no net) -> Net-(J102-Pad21)
- J102 pad 22: (no net) -> Net-(J102-Pad22)
- J102 pad 23: (no net) -> Net-(J102-Pad23)
- J102 pad 24: (no net) -> Net-(J102-Pad24)
- J102 pad 25: (no net) -> Net-(J102-Pad25)
- J102 pad 26: (no net) -> Net-(J102-Pad26)
- J102 pad 27: (no net) -> Net-(J102-Pad27)
- J102 pad 28: (no net) -> Net-(J102-Pad28)
- J102 pad 29: (no net) -> Net-(J102-Pad29)
- J102 pad 30: (no net) -> Net-(J102-Pad30)
- J103 pad 35: (no net) -> Net-(J103-Pad35)
- J103 pad 37: (no net) -> Net-(J103-Pad37)
- U101 pad 11: (no net) -> ADC-RESET
- U101 pad 2: (no net) -> Net-(U101-Pad2)
- U101 pad 20: (no net) -> Net-(U101-Pad20)
- U101 pad 21: (no net) -> Net-(U101-Pad21)
- U101 pad 22: (no net) -> Net-(U101-Pad22)
- U101 pad 26: (no net) -> Net-(U101-Pad26)
- U101 pad 27: (no net) -> Net-(U101-Pad27)
- U101 pad 28: (no net) -> Net-(U101-Pad28)
- U101 pad 3: (no net) -> Net-(U101-Pad3)
- U101 pad 34: (no net) -> Net-(U101-Pad34)
- U101 pad 37: (no net) -> Net-(U101-Pad37)
- U101 pad 4: (no net) -> Net-(U101-Pad4)
- U101 pad 42: (no net) -> Net-(U101-Pad42)
- U101 pad 43: (no net) -> Net-(U101-Pad43)
- U101 pad 46: (no net) -> Net-(U101-Pad46)
- U101 pad 7: (no net) -> Net-(U101-Pad7)
- U104 pad 7: (no net) -> Net-(U104-Pad7)
- U104 pad 8: (no net) -> Net-(U104-Pad8)
- U106 pad 12: (no net) -> Net-(U106-Pad12)
- U106 pad 2: (no net) -> Net-(U106-Pad2)
- U201 pad 16: (no net) -> Net-(U201-Pad16)
- U201 pad 18: (no net) -> Net-(U201-Pad18)
- U201 pad 20: (no net) -> Net-(U201-Pad20)
- U202 pad 16: (no net) -> Net-(U202-Pad16)
- U202 pad 18: (no net) -> Net-(U202-Pad18)
- U202 pad 20: (no net) -> Net-(U202-Pad20)
- U204 pad 16: (no net) -> Net-(U204-Pad16)
- U204 pad 18: (no net) -> Net-(U204-Pad18)
- U204 pad 20: (no net) -> Net-(U204-Pad20)
- U205 pad 16: (no net) -> Net-(U205-Pad16)
- U205 pad 18: (no net) -> Net-(U205-Pad18)
- U205 pad 20: (no net) -> Net-(U205-Pad20)
- U207 pad 7: (no net) -> Net-(U207-Pad7)
- U208 pad 3: (no net) -> Net-(U208-Pad3)
- U208 pad 7: (no net) -> Net-(U208-Pad7)
- U209 pad 1: (no net) -> Net-(U209-Pad1)
- U209 pad 12: (no net) -> Net-(U209-Pad12)
- U209 pad 3: (no net) -> Net-(U209-Pad3)

Commit message: fix isolator enable resistors
Parts:
- R221, R254: value 4.7k -> 0

Commit message: fix diodes
Parts:
- D201, D202, D213, D214, D217, D218, D221, D222: value SMBJ18A -> SMBJ18CA

Commit message: add version 1,1
fix footprints
Parts:
- C111: value TBD -> 100µF/35V; footprint kicad-libraries:ELKO_83 -> kicad-libraries:ELKO_63
- C122, C123, C124: footprint kicad-libraries:ELKO_83 -> kicad-libraries:ELKO_63
- C205, C206, C223, C224: footprint kicad-libraries:C0603F -> kicad-libraries:C0402F
- C239, C242: value 2.2uF/30V -> 4.7uF/30V
- R109: footprint kicad-libraries:R0603F -> kicad-libraries:R0402F
- moved C124 1.00 mm to (160.8, 117.6)
- moved C122 1.00 mm to (169.7, 117.6)
- moved C123 0.73 mm to (161.4, 134.5)
- moved C111 0.68 mm to (165.3, 90.1)
- moved R109 0.68 mm to (175.4, 105.7)
- moved C206 0.35 mm to (106.0, 105.6)
- moved C223 0.35 mm to (106.0, 121.6)
- moved C224 0.32 mm to (106.0, 137.6)
- moved C205 0.30 mm to (106.0, 89.7)
Routing:
- added copper zone on F.Cu, net (none)
- added copper zone on F.Cu, net AGND
- added copper zone on F.Cu, net AGNDA
Other:
- board text added: "Copyright Tinkerforge GmbH 2020. This documentation describes Open Hardware and is licensed under the CERN OHL v. 1.1. You may redistribute and modify this documentation under the terms of the CERN OHL v.1.1. (http://ohwr.org/cernohl). This documentation is distributed WITHOUT ANY EXPRESS OR IMPLIED WARRANTY, INCLUDING OF MERCHANTABILITY, SATISFACTORY QUALITY AND FITNESS FOR A PARTICULAR PURPOSE.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"

Commit message: fix text layer
Routing:
- removed copper zone on F.Cu, net (none)
